File: hardware/qsd/qsd.sch (KiCad schematic (older format))
At the start: 44 parts, among them J1 Conn_01x02, J2 Conn_01x02, J3 Conn_01x02, J4 Conn_01x02, J5 Conn_01x02, U1 MCP6476UT-E_OT, U2 74LS163, U3 MCP6476UT-E_OT, U4 SN74CBT3253, U5 MCP6476UT-E_OT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

Commit message: add schematics
Parts:
- added C17, C18: 1u, Capacitor_SMD:C_1206_3216Metric, symbol Device:C_Small
- R4: value 10k -> 100
- RV1: footprint (none) -> Connector_PinHeader_2.54mm:PinHeader_1x03_P2.54mm_Vertical
Connections:
- net +5V: no longer R4.1
- net GND: now also C18.1; no longer R5.2
- net Vref: now also R4.2
- net at C3.1, R5.1, U2.2 (CP): no longer R4.2
- net at R1.2, RV1.1, RV1.2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: now also C17.2
- net at R7.1, RV1.3, U3.4 (-): now also C17.1
- new net: C18.2, R4.1, R5.2
Other:
- moved on the sheet: R4, R8
Changed lines of the file:
@@
 	2050 2300 2050 2000
-Wire Wire Line
-	2050 900  2650 900
-Wire Wire Line
-	2650 900  2650 1000
 Wire Wire Line
 	2150 1300 2050 1300
@@
 	1    0    0    -1
 $EndComp
-Wire Wire Line
-	2650 850  2650 900
-Connection ~ 2650 900
-$Comp
-L Device:R_Small R4
-U 1 1 61E92221
-P 1750 1950
-F 0 "R4" H 1809 1996 50  0000 L CNN
-F 1 "10k" H 1809 1905 50  0000 L CNN
-F 2 "Resistor_SMD:R_1206_3216Metric" H 1750 1950 50  0001 C CNN
-F 3 "~" H 1750 1950 50  0001 C CNN
-	1    1750 1950
-	1    0    0    -1
-$EndComp
 $Comp
 L Device:R_Small R5
@@
 $EndComp
 Wire Wire Line
-	1750 2050 1750 2100
-Wire Wire Line
 	1750 2100 2150 2100
 Connection ~ 1750 2100
@@
 Wire Wire Line
 	2650 2650 2650 2600
-$Comp
-L power:GND #PWR0103
-U 1 1 61E9450A
-P 1750 2400
-F 0 "#PWR0103" H 1750 2150 50  0001 C CNN
-F 1 "GND" H 1755 2227 50  0000 C CNN
-F 2 "" H 1750 2400 50  0001 C CNN
-F 3 "" H 1750 2400 50  0001 C CNN
-	1    1750 2400
-	1    0    0    -1
-$EndComp
-Wire Wire Line
-	1750 2400 1750 2350
 $Comp
 L Device:C_Small C3
@@
 Wire Wire Line
 	1600 2100 1750 2100
-Wire Wire Line
-	1750 1850 1750 1800
-$Comp
-L power:+5V #PWR0104
-U 1 1 61E96F67
-P 1750 1800
-F 0 "#PWR0104" H 1750 1650 50  0001 C CNN
-F 1 "+5V" H 1765 1973 50  0000 C CNN
-F 2 "" H 1750 1800 50  0001 C CNN
-F 3 "" H 1750 1800 50  0001 C CNN
-	1    1750 1800
-	1    0    0    -1
-$EndComp
 $Comp
 L Connector_Generic:Conn_01x02 J2
@@
 U 1 1 61ED12CA
 P 2400 4000
-F 0 "R7" V 2500 3900 50  0000 C CNN
-F 1 "1k" V 2500 4050 50  0000 C CNN
+F 0 "R7" V 2300 4000 50  0000 C CNN
+F 1 "1k" V 2350 3850 50  0000 C CNN
 F 2 "Resistor_SMD:R_1206_3216Metric" H 2400 4000 50  0001 C CNN
 F 3 "~" H 2400 4000 50  0001 C CNN
@@
 U 1 1 61ED849D
 P 2200 3500
-F 0 "C7" H 2108 3454 50  0000 R CNN
+F 0 "C7" H 2150 3450 50  0000 R CNN
 F 1 "1u" H 2108 3545 50  0000 R CNN
 F 2 "Capacitor_SMD:C_1206_3216Metric" H 2200 3500 50  0001 C CNN
@@
 U 1 1 61EF26A6
 P 2900 4550
-F 0 "RV1" V 2950 4350 50  0000 C CNN
-F 1 "100k" V 3000 4350 50  0000 C CNN
-F 2 "" H 2900 4550 50  0001 C CNN
+F 0 "RV1" V 2850 4300 50  0000 C CNN
+F 1 "100k" V 2950 4300 50  0000 C CNN
+F 2 "Connector_PinHeader_2.54mm:PinHeader_1x03_P2.54mm_Vertical" H 2900 4550 50  0001 C CNN
 F 3 "~" H 2900 4550 50  0001 C CNN
 	1    2900 4550
@@
 U 1 1 61EFF79A
 P 1650 4000
-F 0 "C4" V 1879 4000 50  0000 C CNN
-F 1 "1u" V 1788 4000 50  0000 C CNN
+F 0 "C4" V 1800 4100 50  0000 C CNN
+F 1 "1u" V 1800 3950 50  0000 C CNN
 F 2 "Capacitor_SMD:C_1206_3216Metric" H 1650 4000 50  0001 C CNN
 F 3 "~" H 1650 4000 50  0001 C CNN
@@
 Wire Wire Line
 	1100 4100 1100 4150
-Text GLabel 2650 5700 2    50   Input ~ 0
+Text GLabel 2900 5700 2    50   Input ~ 0
 Vref
 $Comp
 L Device:R_Small R8
 U 1 1 61F0D5B8
-P 2500 5700
-F 0 "R8" V 2304 5700 50  0000 C CNN
-F 1 "100" V 2395 5700 50  0000 C CNN
-F 2 "Resistor_SMD:R_1206_3216Metric" H 2500 5700 50  0001 C CNN
-F 3 "~" H 2500 5700 50  0001 C CNN
-	1    2500 5700
+P 2650 5700
+F 0 "R8" V 2550 5700 50  0000 C CNN
+F 1 "100" V 2750 5700 50  0000 C CNN
+F 2 "Resistor_SMD:R_1206_3216Metric" H 2650 5700 50  0001 C CNN
+F 3 "~" H 2650 5700 50  0001 C CNN
+	1    2650 5700
 	0    1    1    0
 $EndComp
@@
 Wire Wire Line
 	2350 5700 2300 5700
-Wire Wire Line
-	2400 5700 2350 5700
 Connection ~ 2350 5700
-Wire Wire Line
-	2650 5700 2600 5700
 $Comp
 L Device:R_Small R2
@@
 U 1 1 61F9B74D
 P 5450 4800
-F 0 "C11" H 5358 4754 50  0000 R CNN
+F 0 "C11" H 5400 4750 50  0000 R CNN
 F 1 "1u" H 5358 4845 50  0000 R CNN
 F 2 "Capacitor_SMD:C_1206_3216Metric" H 5450 4800 50  0001 C CNN
@@
 U 1 1 61F9BEAE
 P 5750 4800
-F 0 "C12" H 5658 4754 50  0000 R CNN
+F 0 "C12" H 5700 4750 50  0000 R CNN
 F 1 "1u" H 5658 4845 50  0000 R CNN
 F 2 "Capacitor_SMD:C_1206_3216Metric" H 5750 4800 50  0001 C CNN
@@
 U 1 1 61F9D549
 P 6050 4800
-F 0 "C13" H 5958 4754 50  0000 R CNN
+F 0 "C13" H 6000 4750 50  0000 R CNN
 F 1 "1u" H 5958 4845 50  0000 R CNN
 F 2 "Capacitor_SMD:C_1206_3216Metric" H 6050 4800 50  0001 C CNN
@@
 U 1 1 61F9D9B4
 P 6350 4800
-F 0 "C14" H 6258 4754 50  0000 R CNN
+F 0 "C14" H 6300 4750 50  0000 R CNN
 F 1 "1u" H 6258 4845 50  0000 R CNN
 F 2 "Capacitor_SMD:C_1206_3216Metric" H 6350 4800 50  0001 C CNN
@@
 U 1 1 62057D83
 P 7450 3850
-F 0 "R11" V 7350 3800 50  0000 C CNN
-F 1 "10k" V 7350 3950 50  0000 C CNN
+F 0 "R11" V 7350 3850 50  0000 C CNN
+F 1 "10k" V 7400 3700 50  0000 C CNN
 F 2 "Resistor_SMD:R_1206_3216Metric" H 7450 3850 50  0001 C CNN
 F 3 "~" H 7450 3850 50  0001 C CNN
@@
 U 1 1 62057D8D
 P 7450 4050
-F 0 "R12" V 7350 4100 50  0000 C CNN
-F 1 "10k" V 7350 3950 50  0000 C CNN
+F 0 "R12" V 7550 4050 50  0000 C CNN
+F 1 "10k" V 7500 4200 50  0000 C CNN
 F 2 "Resistor_SMD:R_1206_3216Metric" H 7450 4050 50  0001 C CNN
 F 3 "~" H 7450 4050 50  0001 C CNN
@@
 U 1 1 62057DCC
 P 8000 4850
-F 0 "C16" V 7850 4800 50  0000 C CNN
+F 0 "C16" V 7850 4700 50  0000 C CNN
 F 1 "1u" V 7850 4900 50  0000 C CNN
 F 2 "Capacitor_SMD:C_1206_3216Metric" H 8000 4850 50  0001 C CNN
@@
 Wire Wire Line
 	1650 7150 1950 7150
+Wire Wire Line
+	2350 5700 2550 5700
+Wire Wire Line
+	2750 5700 2900 5700
+$Comp
+L Device:C_Small C17
+U 1 1 6222DB4B
+P 2900 4900
+F 0 "C17" H 2850 4850 50  0000 R CNN
+F 1 "1u" H 2808 4945 50  0000 R CNN
+F 2 "Capacitor_SMD:C_1206_3216Metric" H 2900 4900 50  0001 C CNN
+F 3 "~" H 2900 4900 50  0001 C CNN
+	1    2900 4900
+	0    -1   -1   0
+$EndComp
+Wire Wire Line
+	2800 4900 2550 4900
+Wire Wire Line
+	2550 4900 2550 4550
+Connection ~ 2550 4550
+Wire Wire Line
+	3000 4900 3300 4900
+Wire Wire Line
+	3300 4900 3300 4550
+Connection ~ 3300 4550
+$Comp
+L Device:R_Small R4
+U 1 1 61E92221
+P 1600 2450
+F 0 "R4" V 1404 2450 50  0000 C CNN
+F 1 "100" V 1495 2450 50  0000 C CNN
+F 2 "Resistor_SMD:R_1206_3216Metric" H 1600 2450 50  0001 C CNN
+F 3 "~" H 1600 2450 50  0001 C CNN
+	1    1600 2450
+	0    1    1    0
+$EndComp
+Wire Wire Line
+	1700 2450 1750 2450
+Wire Wire Line
+	1750 2350 1750 2450
+$Comp
+L Device:C_Small C18
+U 1 1 6226B7C4
+P 1750 2600
+F 0 "C18" H 1700 2550 50  0000 R CNN
+F 1 "1u" H 1658 2645 50  0000 R CNN
+F 2 "Capacitor_SMD:C_1206_3216Metric" H 1750 2600 50  0001 C CNN
+F 3 "~" H 1750 2600 50  0001 C CNN
+	1    1750 2600
+	-1   0    0    1
+$EndComp
+Wire Wire Line
+	1750 2500 1750 2450
+Connection ~ 1750 2450
+$Comp
+L power:GND #PWR0103
+U 1 1 62277A73
+P 1750 2750
+F 0 "#PWR0103" H 1750 2500 50  0001 C CNN
+F 1 "GND" H 1755 2577 50  0000 C CNN
+F 2 "" H 1750 2750 50  0001 C CNN
+F 3 "" H 1750 2750 50  0001 C CNN
+	1    1750 2750
+	1    0    0    -1
+$EndComp
+Wire Wire Line
+	1750 2750 1750 2700
+Text GLabel 1450 2450 0    50   Input ~ 0
+Vref
+Wire Wire Line
+	1450 2450 1500 2450
+Wire Wire Line
+	2650 850  2650 900
+Wire Wire Line
+	2650 900  2650 1000
+Connection ~ 2650 900
+Wire Wire Line
+	2050 900  2650 900
 $EndSCHEMATC
